File: cryptick-token-pcb.kicad_sch (KiCad schematic)
At the start: 14 parts, among them J1 Conn_02x08_Counter_Clockwise, J2 Conn_02x08_Counter_Clockwise, J3 OLED DISPLAY, J4 Encoder, J5 Conn_01x09, J6 Conn_01x09, J7 Fingerprint_Sensor, SW1 SW_DPST, SW2 SW_DPST, SW3 SW_DPST, U1 ESP32-S3-WROOM-1

Commit message: late release
Parts:
- removed J1, J2: Conn_02x08_Counter_Clockwise, Connector_PinHeader_2.54mm:PinHeader_2x08_P2.54mm_Vertical, symbol Connector_Generic:Conn_02x08_Counter_Clockwise
- removed J4: Encoder, symbol Connector:Conn_01x05_Socket
- removed J5, J6: Conn_01x09, symbol Connector_Generic:Conn_01x09
- removed SW1, SW2, SW3: SW_DPST, symbol Switch:SW_DPST
- added B1: CR2032-BS-6-1, easyeda2kicad:BAT-TH_CR2032-BS-6-1, symbol easyeda2kicad:CR2032-BS-6-1
- added BT1: BS-12-A1AJ002-F, easyeda2kicad:BAT-TH_BS-12-A1AJ002-F, symbol easyeda2kicad:BS-12-A1AJ002-F
- added C1, C4: 22u, Capacitor_SMD:C_0805_2012Metric, symbol Device:C
- added C10, C2, C9: 1u, Capacitor_SMD:C_0805_2012Metric, symbol Device:C
- added C3, C7, C8: 10u, Capacitor_SMD:C_0805_2012Metric, symbol Device:C
- added C5: 100n, Capacitor_SMD:C_0603_1608Metric, symbol Device:C
- added C6: 33p, Capacitor_SMD:C_0603_1608Metric, symbol Device:C
- added CN1: YXT-BB10-24S-02, easyeda2kicad:CONN-SMD_YXT-BB10-24S-02, symbol easyeda2kicad:YXT-BB10-24S-02
- added CN2: SM02B-SRSS-TB, easyeda2kicad:CONN-SMD_2P-P1.00_SM02B-SRSS-TB-LF-SN, symbol easyeda2kicad:SM02B-SRSS-TB
- added D1: 5V, LED_SMD:LED_0603_1608Metric, symbol Device:LED
- added D2: PTVS5V0S1UR, Diode_SMD:D_SOD-123, symbol Diode:PTVS5V0Z1USK
- added FPC1: FPC-05F-20PH20, easyeda2kicad:FPC-SMD_20P-P0.50_XUNPU_FPC-05F-20PH20, symbol easyeda2kicad:FPC-05F-20PH20
- added H1, H2: MountingHole_Pad, MountingHole:MountingHole_2.2mm_M2_Pad_Via, symbol Mechanical:MountingHole_Pad
- added J1: USB_C_Receptacle_USB2.0_16P, Connector_USB:USB_C_Receptacle_G-Switch_GT-USB-7010ASV, symbol Connector:USB_C_Receptacle_USB2.0_16P
- added J5: JST-6 PIN-JST-SH, Connector_JST:JST_SH_BM06B-SRSS-TB_1x06-1MP_P1.00mm_Vertical, symbol Connector:Conn_01x06_Socket
- added Q1: AO3400A, Package_TO_SOT_SMD:SOT-23, symbol Transistor_FET_Other:Q_NMOS_Depletion_GSD
- added R10, R20, R21, R4, R5, R6, R7, R8: 10K, Resistor_SMD:R_0603_1608Metric, symbol Device:R
- added R11: 10R, Resistor_SMD:R_0603_1608Metric, symbol Device:R
- added R12, R13: 5K1, Resistor_SMD:R_0603_1608Metric, symbol Device:R
- added R14, R15, R17, R19: 1K, Resistor_SMD:R_0603_1608Metric, symbol Device:R
- added R16, R18: 22R, Resistor_SMD:R_0603_1608Metric, symbol Device:R
- added R9: 100R, Resistor_SMD:R_0603_1608Metric, symbol Device:R
- added SW1: K1-5202UA-01, easyeda2kicad:SW-SMD_K1-5202UA-01, symbol easyeda2kicad:K1-5202UA-01
- added SW2: EC05E1220401, easyeda2kicad:SW-SMD_EC05E1220401, symbol easyeda2kicad:EC05E1220401
- added SW3: MSK12C02-HB, easyeda2kicad:SW-TH_MSK12C02-HB-1, symbol easyeda2kicad:MSK12C02-HB
- added U1: DS3231MZ, Package_SO:SOIC-8_3.9x4.9mm_P1.27mm, symbol Timer_RTC:DS3231MZ
- added U3: ME6217C33M5G, easyeda2kicad:SOT-23-5_L3.0-W1.7-P0.95-LS2.8-BR, symbol easyeda2kicad:ME6217C33M5G
- added U4: BQ25185DLHR, easyeda2kicad:WSON-10_L2.2-W2.0-P0.40-BL-EP_TI_DLH0010A, symbol easyeda2kicad:BQ25185DLHR
- added U5: USBLC6-2SC6, Package_TO_SOT_SMD:SOT-23-6, symbol Power_Protection:USBLC6-2SC6
- J3: footprint (none) -> Connector_PinHeader_2.54mm:PinHeader_1x04_P2.54mm_Vertical
- J4: renamed from J7; footprint (none) -> Connector_JST:JST_SH_BM06B-SRSS-TB_1x06-1MP_P1.00mm_Vertical; ID (none) -> C2904988; MPN (none) -> 1.0-6PS; Manufacturer (none) -> DEALON
- R1, R2, R3: value R -> 10K; footprint (none) -> Resistor_SMD:R_0603_1608Metric; ID (none) -> C98220; MPN (none) -> RC0603FR-0710KL; Manufacturer (none) -> YAGEO
- renumbered U1 to U2
Connections:
- net VCC is gone; now on net +3V3: J3.2 (Pin_2)
- net +3V3: now also R1.2, R2.1, R3.1, U2.2 (3V3), C2.1, C4.1, C5.1, C6.1, C7.1, CN1.1, CN1.17, CN1.2, FPC1.12, FPC1.8, J5.4 (Pin_4), R20.2, R21.2, R4.1, R5.1, R6.1, R7.1, R8.1, U1.2 (VCC), U3.5 (VOUT)
- net +5V: now also C3.1, SW3.2, U3.1 (VIN), U3.3 (CE)
- net EN: now also R1.1, U2.3 (EN), C1.1, J5.1 (Pin_1)
- net GND: now also BT1.2, C1.2, C10.2, C2.2, C3.2, C4.2, C5.2, C6.2, C7.2, C8.2, C9.2, CN1.19, CN1.22, CN1.25, CN1.26, CN1.27, CN1.28, CN1.5, CN1.6, CN1.8, CN2.1, CN2.3, CN2.4, D1.1 (K), D2.2 (A), FPC1.1, FPC1.10, FPC1.17, FPC1.2, FPC1.20, FPC1.21, FPC1.22, FPC1.3, FPC1.9, H1.1, H2.1, J1.A1 (GND), J1.A12 (GND), J1.B1 (GND), J1.B12 (GND), J1.S1 (SHIELD), J5.5 (Pin_5), Q1.2 (S), R10.2, R12.2, R13.2, R15.2, R17.2, R19.2, SW1.5 (COM), SW1.7 (COM), SW1.8 (COM), SW2.4, SW2.5, SW2.C, SW3.4, U1.5 (GND), U3.2 (VSS), U4.11 (EP), U4.4 (~{CE}), U4.5 (GND), U5.2 (GND)
- net SCL: now also U2.17 (IO9), CN1.24, FPC1.6, R21.1, U1.8 (SCL)
- net SDA: now also U2.12 (IO8), CN1.23, FPC1.5, R20.1, U1.7 (SDA)
- net SENSOR_IRQ: now also U2.9 (IO16)
- net SENSOR_RX: now also U2.10 (IO17)
- net SENSOR_TX: now also U2.11 (IO18)
- net USB_D-: now reaches U2.13 (USB_D-)
- net USB_D-: now also R16.2
- net USB_D+: now reaches U2.14 (USB_D+)
- net USB_D+: now also R18.2
- net CS0: now reaches U2.18 (IO10)
- net CS0: now also CN1.10, FPC1.11
- net SDO: now reaches U2.19 (IO11)
- net SDO: now also FPC1.14
- net SCK: now reaches U2.20 (IO12)
- net SCK: now also FPC1.13
- net SDI: now reaches U2.21 (IO13)
- net CS1: now reaches U2.22 (IO14)
- net CS2: now reaches U2.23 (IO21)
- net LCD_RS: now reaches U2.24 (IO47)
- net LCD_RS: now also CN1.14, FPC1.15
- net LCD_RESET: now reaches U2.25 (IO48)
- net LCD_RESET: now also CN1.16, FPC1.16
- net IO0: now reaches U2.27 (IO0)
- net IO0: now also J5.6 (Pin_6)
- net STAT1: now reaches U2.31 (IO38)
- net STAT1: now also U4.9 (STAT1)
- net STAT2: now reaches U2.32 (IO39)
- net STAT2: now also U4.3 (STAT2)
- net CW: now reaches U2.33 (IO40)
- net CW: now also R8.2, SW2.A
- net CCW: now reaches U2.34 (IO41)
- net CCW: now also R7.2, SW2.B
- net LCD_BRIGHTNESS: now reaches U2.35 (IO42)
- net LCD_BRIGHTNESS: now also R9.1
- net RX: now reaches U2.36 (RXD0)
- net RX: now also J5.2 (Pin_2)
- net TX: now reaches U2.37 (TXD0)
- net TX: now also J5.3 (Pin_3)
- net TP_INT: now reaches U2.38 (IO2)
- net TP_INT: now also CN1.20, FPC1.7
- net TP_RESET: now reaches U2.39 (IO1)
- net TP_RESET: now also CN1.21, FPC1.4
- net RIGHT: now reaches U2.4 (IO4)
- net RIGHT: now also R6.2, SW1.4 (RIGHT)
- net DOWN: now reaches U2.5 (IO5)
- net DOWN: now also R5.2, SW1.6 (DOWN)
- net UP: now reaches U2.6 (IO6)
- net UP: now also R2.2, SW1.1 (UP)
- net LEFT: now reaches U2.7 (IO7)
- net LEFT: now also R4.2, SW1.3 (LEFT)
- net CENTER: now reaches U2.8 (IO15)
- net CENTER: now also R3.2, SW1.2 (CENTER)
- new net: Q1.3 (D), R11.2
- new net: Q1.1 (G), R10.1, R9.2
- new net: D1.2 (A), R14.2
- new net: J1.A5 (CC1), R12.1
- new net: J1.B5 (CC2), R13.1
- new net BAT: C9.1, CN2.2, U4.2 (BAT)
- new net D+: R18.1, U5.6 (I/O1)
- new net D-: R16.1, U5.4 (I/O2)
- new net ILIM/VSET: R17.1, U4.7 (ILIM/VSET)
- new net ISET: R19.1, U4.8 (ISET)
- new net LCD_MOSI: CN1.12
- new net LCD_SCLK: CN1.11
- new net LEDA: FPC1.18
- new net LEDK: CN1.3, FPC1.19, R11.1
- new net SYS: C8.1, SW3.3, U4.1 (SYS)
- new net TS/MR: R15.1, U4.6 (TS/MR)
- new net USB_conn+: J1.A6 (D+), J1.B6 (D+), U5.1 (I/O1)
- new net USB_conn-: J1.A7 (D-), J1.B7 (D-), U5.3 (I/O2)
- new net VBAT: BT1.1, U1.6 (VBAT)
- new net VBUS: C10.1, D2.1 (K), J1.A4 (VBUS), J1.A9 (VBUS), J1.B4 (VBUS), J1.B9 (VBUS), R14.1, U4.10 (IN), U5.5 (VBUS)
- no-connect marks 0 -> 20
Other:
- removed sheet documents
- note added: "1U is recommended for snappy boot time by esp guide."
- note added: "AAA-BAT-046-K01"
- note added: "C2926854"
- note added: "Mirrror Vertically (Y) As the Pinout is Flipped in the LCD Connector."
- note added: "Strapping Pins"
- note added: "U1RXD"
- note added: "U1TXD"
- note added: "for esp-idf defaults #define I2C_MASTER_SDA_IO IO1 #define I2C_MASTER_SCL_IO IO2"
- note added: "https://docs.espressif.com/projects/esp-idf/en/v5.1.5/esp32s3/api-reference/peripherals/spi_master.html"
- note added: "https://oshwa.org/resources/a-resolution-to-redefine-spi-signal-names/"
- note added: "https://yarsa.tech/files/DT80160S096NA-2310BS001.pdf"
- moved on the sheet: J3, J4, U2
